File: himax_usb_board/bus_mux.kicad_sch (KiCad schematic)
At the start: 6 parts

Commit message: board routing wip
Parts:
- C59, C60, C61: renamed from C?; footprint (none) -> Capacitor_SMD:C_0402_1005Metric
- U12, U13, U14: renamed from U?; footprint DHVQFN16_SOT763-1_NEX -> 74CBTLV3257BQ_115:DHVQFN16_SOT763-1_NEX
Connections:
- no-connect marks 0 -> 1
Changed lines of the file:
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@@
   (junction (at 116.84 157.48) (diameter 0) (color 0 0 0 0)
   )
+  (no_connect (at 119.38 149.86))
   (bus_entry (at 97.79 97.79) (size 2.54 2.54)
     (stroke (width 0) (type default) (color 0 0 0 0))
@@
   (symbol (lib_id "74CBTLV3257BQ_115:74CBTLV3257BQ_115") (at 127 127 0) (unit 1)
     (in_bom yes) (on_board yes) (fields_autoplaced)
-    (property "Reference" "U?" (id 0) (at 139.7 122.8524 0)
+    (property "Reference" "U14" (id 0) (at 139.7 122.8524 0)
       (effects (font (size 1.524 1.524)))
     )
@@
       (effects (font (size 1.524 1.524)))
     )
-    (property "Footprint" "DHVQFN16_SOT763-1_NEX" (id 2) (at 105.41 120.65 0)
+    (property "Footprint" "74CBTLV3257BQ_115:DHVQFN16_SOT763-1_NEX" (id 2) (at 105.41 120.65 0)
       (effects (font (size 1.27 1.27) italic) hide)
     )
@@
   (symbol (lib_id "power:GND") (at 160.02 97.79 90) (mirror x) (unit 1)
     (in_bom yes) (on_board yes) (fields_autoplaced)
-    (property "Reference" "#PWR?" (id 0) (at 166.37 97.79 0)
+    (property "Reference" "#PWR0144" (id 0) (at 166.37 97.79 0)
       (effects (font (size 1.27 1.27)) hide)
     )
@@
   (symbol (lib_id "power:+2V8") (at 111.76 30.48 0) (unit 1)
     (in_bom yes) (on_board yes)
-    (property "Reference" "#PWR?" (id 0) (at 111.76 34.29 0)
+    (property "Reference" "#PWR0132" (id 0) (at 111.76 34.29 0)
       (effects (font (size 1.27 1.27)) hide)
     )
@@
   (symbol (lib_id "power:GND") (at 119.38 134.62 270) (unit 1)
     (in_bom yes) (on_board yes)
-    (property "Reference" "#PWR?" (id 0) (at 113.03 134.62 0)
+    (property "Reference" "#PWR0140" (id 0) (at 113.03 134.62 0)
       (effects (font (size 1.27 1.27)) hide)
     )
@@
   (symbol (lib_id "power:GND") (at 116.84 71.12 0) (mirror y) (unit 1)
     (in_bom yes) (on_board yes) (fields_autoplaced)
-    (property "Reference" "#PWR?" (id 0) (at 116.84 77.47 0)
+    (property "Reference" "#PWR0135" (id 0) (at 116.84 77.47 0)
       (effects (font (size 1.27 1.27)) hide)
     )
@@
   (symbol (lib_id "power:GND") (at 160.02 149.86 90) (mirror x) (unit 1)
     (in_bom yes) (on_board yes) (fields_autoplaced)
-    (property "Reference" "#PWR?" (id 0) (at 166.37 149.86 0)
+    (property "Reference" "#PWR0146" (id 0) (at 166.37 149.86 0)
       (effects (font (size 1.27 1.27)) hide)
     )
@@
   (symbol (lib_id "power:GND") (at 160.02 58.42 90) (mirror x) (unit 1)
     (in_bom yes) (on_board yes) (fields_autoplaced)
-    (property "Reference" "#PWR?" (id 0) (at 166.37 58.42 0)
+    (property "Reference" "#PWR0142" (id 0) (at 166.37 58.42 0)
       (effects (font (size 1.27 1.27)) hide)
     )
@@
   (symbol (lib_id "power:GND") (at 116.84 160.02 0) (mirror y) (unit 1)
     (in_bom yes) (on_board yes) (fields_autoplaced)
-    (property "Reference" "#PWR?" (id 0) (at 116.84 166.37 0)
+    (property "Reference" "#PWR0137" (id 0) (at 116.84 166.37 0)
       (effects (font (size 1.27 1.27)) hide)
     )
@@
   (symbol (lib_id "power:GND") (at 116.84 115.57 0) (mirror y) (unit 1)
     (in_bom yes) (on_board yes) (fields_autoplaced)
-    (property "Reference" "#PWR?" (id 0) (at 116.84 121.92 0)
+    (property "Reference" "#PWR0136" (id 0) (at 116.84 121.92 0)
       (effects (font (size 1.27 1.27)) hide)
     )
@@
   (symbol (lib_id "74CBTLV3257BQ_115:74CBTLV3257BQ_115") (at 127 38.1 0) (unit 1)
     (in_bom yes) (on_board yes) (fields_autoplaced)
-    (property "Reference" "U?" (id 0) (at 139.7 33.9524 0)
+    (property "Reference" "U12" (id 0) (at 139.7 33.9524 0)
       (effects (font (size 1.524 1.524)))
     )
@@
       (effects (font (size 1.524 1.524)))
     )
-    (property "Footprint" "DHVQFN16_SOT763-1_NEX" (id 2) (at 105.41 31.75 0)
+    (property "Footprint" "74CBTLV3257BQ_115:DHVQFN16_SOT763-1_NEX" (id 2) (at 105.41 31.75 0)
       (effects (font (size 1.27 1.27) italic) hide)
     )
@@
   (symbol (lib_id "Device:C_Small") (at 109.22 124.46 0) (mirror x) (unit 1)
     (in_bom yes) (on_board yes) (fields_autoplaced)
-    (property "Reference" "C?" (id 0) (at 106.8959 123.6189 0)
+    (property "Reference" "C61" (id 0) (at 106.8959 123.6189 0)
       (effects (font (size 1.27 1.27)) (justify right))
     )
@@
       (effects (font (size 1.27 1.27)) (justify right))
     )
-    (property "Footprint" "" (id 2) (at 109.22 124.46 0)
+    (property "Footprint" "Capacitor_SMD:C_0402_1005Metric" (id 2) (at 109.22 124.46 0)
       (effects (font (size 1.27 1.27)) hide)
     )
@@
   (symbol (lib_id "power:GND") (at 109.22 127 0) (unit 1)
     (in_bom yes) (on_board yes)
-    (property "Reference" "#PWR?" (id 0) (at 109.22 133.35 0)
+    (property "Reference" "#PWR0131" (id 0) (at 109.22 133.35 0)
       (effects (font (size 1.27 1.27)) hide)
     )
@@
   (symbol (lib_id "power:GND") (at 119.38 45.72 270) (unit 1)
     (in_bom yes) (on_board yes)
-    (property "Reference" "#PWR?" (id 0) (at 113.03 45.72 0)
+    (property "Reference" "#PWR0138" (id 0) (at 113.03 45.72 0)
       (effects (font (size 1.27 1.27)) hide)
     )
@@
   (symbol (lib_id "power:GND") (at 109.22 82.55 0) (unit 1)
     (in_bom yes) (on_board yes)
-    (property "Reference" "#PWR?" (id 0) (at 109.22 88.9 0)
+    (property "Reference" "#PWR0130" (id 0) (at 109.22 88.9 0)
       (effects (font (size 1.27 1.27)) hide)
     )
@@
   (symbol (lib_id "power:GND") (at 160.02 137.16 90) (mirror x) (unit 1)
     (in_bom yes) (on_board yes) (fields_autoplaced)
-    (property "Reference" "#PWR?" (id 0) (at 166.37 137.16 0)
+    (property "Reference" "#PWR0145" (id 0) (at 166.37 137.16 0)
       (effects (font (size 1.27 1.27)) hide)
     )
@@
   (symbol (lib_id "74CBTLV3257BQ_115:74CBTLV3257BQ_115") (at 127 82.55 0) (unit 1)
     (in_bom yes) (on_board yes) (fields_autoplaced)
-    (property "Reference" "U?" (id 0) (at 139.7 78.4024 0)
+    (property "Reference" "U13" (id 0) (at 139.7 78.4024 0)
       (effects (font (size 1.524 1.524)))
     )
@@
       (effects (font (size 1.524 1.524)))
     )
-    (property "Footprint" "DHVQFN16_SOT763-1_NEX" (id 2) (at 105.41 76.2 0)
+    (property "Footprint" "74CBTLV3257BQ_115:DHVQFN16_SOT763-1_NEX" (id 2) (at 105.41 76.2 0)
       (effects (font (size 1.27 1.27) italic) hide)
     )
@@
   (symbol (lib_id "power:+2V8") (at 111.76 74.93 0) (unit 1)
     (in_bom yes) (on_board yes)
-    (property "Reference" "#PWR?" (id 0) (at 111.76 78.74 0)
+    (property "Reference" "#PWR0133" (id 0) (at 111.76 78.74 0)
       (effects (font (size 1.27 1.27)) hide)
     )
@@
   (symbol (lib_id "Device:C_Small") (at 109.22 80.01 0) (mirror x) (unit 1)
     (in_bom yes) (on_board yes) (fields_autoplaced)
-    (property "Reference" "C?" (id 0) (at 106.8959 79.1689 0)
+    (property "Reference" "C60" (id 0) (at 106.8959 79.1689 0)
       (effects (font (size 1.27 1.27)) (justify right))
     )
@@
       (effects (font (size 1.27 1.27)) (justify right))
     )
-    (property "Footprint" "" (id 2) (at 109.22 80.01 0)
+    (property "Footprint" "Capacitor_SMD:C_0402_1005Metric" (id 2) (at 109.22 80.01 0)
       (effects (font (size 1.27 1.27)) hide)
     )
@@
   (symbol (lib_id "power:GND") (at 160.02 55.88 90) (mirror x) (unit 1)
     (in_bom yes) (on_board yes) (fields_autoplaced)
-    (property "Reference" "#PWR?" (id 0) (at 166.37 55.88 0)
+    (property "Reference" "#PWR0141" (id 0) (at 166.37 55.88 0)
       (effects (font (size 1.27 1.27)) hide)
     )
@@
   (symbol (lib_id "Device:C_Small") (at 109.22 35.56 0) (mirror x) (unit 1)
     (in_bom yes) (on_board yes) (fields_autoplaced)
-    (property "Reference" "C?" (id 0) (at 106.8959 34.7189 0)
+    (property "Reference" "C59" (id 0) (at 106.8959 34.7189 0)
       (effects (font (size 1.27 1.27)) (justify right))
     )
@@
       (effects (font (size 1.27 1.27)) (justify right))
     )
-    (property "Footprint" "" (id 2) (at 109.22 35.56 0)
+    (property "Footprint" "Capacitor_SMD:C_0402_1005Metric" (id 2) (at 109.22 35.56 0)
       (effects (font (size 1.27 1.27)) hide)
     )
@@
   (symbol (lib_id "power:GND") (at 160.02 60.96 90) (mirror x) (unit 1)
     (in_bom yes) (on_board yes) (fields_autoplaced)
-    (property "Reference" "#PWR?" (id 0) (at 166.37 60.96 0)
+    (property "Reference" "#PWR0143" (id 0) (at 166.37 60.96 0)
       (effects (font (size 1.27 1.27)) hide)
     )
@@
   (symbol (lib_id "power:GND") (at 119.38 90.17 270) (unit 1)
     (in_bom yes) (on_board yes)
-    (property "Reference" "#PWR?" (id 0) (at 113.03 90.17 0)
+    (property "Reference" "#PWR0139" (id 0) (at 113.03 90.17 0)
       (effects (font (size 1.27 1.27)) hide)
     )
@@
   (symbol (lib_id "power:+2V8") (at 111.76 119.38 0) (unit 1)
     (in_bom yes) (on_board yes)
-    (property "Reference" "#PWR?" (id 0) (at 111.76 123.19 0)
+    (property "Reference" "#PWR0134" (id 0) (at 111.76 123.19 0)
       (effects (font (size 1.27 1.27)) hide)
     )
@@
   (symbol (lib_id "power:GND") (at 109.22 38.1 0) (unit 1)
     (in_bom yes) (on_board yes)
-    (property "Reference" "#PWR?" (id 0) (at 109.22 44.45 0)
-      (effects (font (size 1.27 1.27)) hide)
-    )
+    (property "Reference" "#PWR0129" (id 0) (at 109.22 44.45 0)
+      (effects (font (size 1.27 1.27)) hide)
+    )

Commit message: hardware wip
Parts:
- C59, C60, C61: MFR (none) -> Samsung; MFR_PN (none) -> CL05B104KP5NNNC
- U12, U13, U14: MFR (none) -> Nexperia USA; MFR_PN (none) -> 74CBTLV3257BQ,115
Changed lines of the file:
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@@
       (effects (font (size 1.27 1.27) italic) hide)
+    )
+    (property "MFR" "Nexperia USA" (id 4) (at 127 127 0)
+      (effects (font (size 1.27 1.27)) hide)
+    )
+    (property "MFR_PN" "74CBTLV3257BQ,115" (id 5) (at 127 127 0)
+      (effects (font (size 1.27 1.27)) hide)
     )
     (pin "1")
@@
   (symbol (lib_id "power:GND") (at 160.02 97.79 90) (mirror x) (unit 1)
     (in_bom yes) (on_board yes) (fields_autoplaced)
-    (property "Reference" "#PWR0144" (id 0) (at 166.37 97.79 0)
+    (property "Reference" "#PWR0146" (id 0) (at 166.37 97.79 0)
       (effects (font (size 1.27 1.27)) hide)
     )
@@
   (symbol (lib_id "power:+2V8") (at 111.76 30.48 0) (unit 1)
     (in_bom yes) (on_board yes)
-    (property "Reference" "#PWR0132" (id 0) (at 111.76 34.29 0)
+    (property "Reference" "#PWR0134" (id 0) (at 111.76 34.29 0)
       (effects (font (size 1.27 1.27)) hide)
     )
@@
   (symbol (lib_id "power:GND") (at 119.38 134.62 270) (unit 1)
     (in_bom yes) (on_board yes)
-    (property "Reference" "#PWR0140" (id 0) (at 113.03 134.62 0)
+    (property "Reference" "#PWR0142" (id 0) (at 113.03 134.62 0)
       (effects (font (size 1.27 1.27)) hide)
     )
@@
   (symbol (lib_id "power:GND") (at 116.84 71.12 0) (mirror y) (unit 1)
     (in_bom yes) (on_board yes) (fields_autoplaced)
-    (property "Reference" "#PWR0135" (id 0) (at 116.84 77.47 0)
+    (property "Reference" "#PWR0137" (id 0) (at 116.84 77.47 0)
       (effects (font (size 1.27 1.27)) hide)
     )
@@
   (symbol (lib_id "power:GND") (at 160.02 149.86 90) (mirror x) (unit 1)
     (in_bom yes) (on_board yes) (fields_autoplaced)
-    (property "Reference" "#PWR0146" (id 0) (at 166.37 149.86 0)
+    (property "Reference" "#PWR0148" (id 0) (at 166.37 149.86 0)
       (effects (font (size 1.27 1.27)) hide)
     )
@@
   (symbol (lib_id "power:GND") (at 160.02 58.42 90) (mirror x) (unit 1)
     (in_bom yes) (on_board yes) (fields_autoplaced)
-    (property "Reference" "#PWR0142" (id 0) (at 166.37 58.42 0)
+    (property "Reference" "#PWR0144" (id 0) (at 166.37 58.42 0)
       (effects (font (size 1.27 1.27)) hide)
     )
@@
   (symbol (lib_id "power:GND") (at 116.84 160.02 0) (mirror y) (unit 1)
     (in_bom yes) (on_board yes) (fields_autoplaced)
-    (property "Reference" "#PWR0137" (id 0) (at 116.84 166.37 0)
+    (property "Reference" "#PWR0139" (id 0) (at 116.84 166.37 0)
       (effects (font (size 1.27 1.27)) hide)
     )
@@
   (symbol (lib_id "power:GND") (at 116.84 115.57 0) (mirror y) (unit 1)
     (in_bom yes) (on_board yes) (fields_autoplaced)
-    (property "Reference" "#PWR0136" (id 0) (at 116.84 121.92 0)
+    (property "Reference" "#PWR0138" (id 0) (at 116.84 121.92 0)
       (effects (font (size 1.27 1.27)) hide)
     )
@@
     (property "Datasheet" "74CBTLV3257BQ_115" (id 3) (at 106.68 31.75 0)
       (effects (font (size 1.27 1.27) italic) hide)
+    )
+    (property "MFR" "Nexperia USA" (id 4) (at 127 38.1 0)
+      (effects (font (size 1.27 1.27)) hide)
+    )
+    (property "MFR_PN" "74CBTLV3257BQ,115" (id 5) (at 127 38.1 0)
+      (effects (font (size 1.27 1.27)) hide)
     )
     (pin "1")
@@
       (effects (font (size 1.27 1.27)) hide)
     )
+    (property "MFR" "Samsung" (id 4) (at 109.22 124.46 0)
+      (effects (font (size 1.27 1.27)) hide)
+    )
+    (property "MFR_PN" "CL05B104KP5NNNC" (id 5) (at 109.22 124.46 0)
+      (effects (font (size 1.27 1.27)) hide)
+    )
     (pin "1")
     (pin "2")
@@
   (symbol (lib_id "power:GND") (at 109.22 127 0) (unit 1)
     (in_bom yes) (on_board yes)
-    (property "Reference" "#PWR0131" (id 0) (at 109.22 133.35 0)
+    (property "Reference" "#PWR0133" (id 0) (at 109.22 133.35 0)
       (effects (font (size 1.27 1.27)) hide)
     )
@@
   (symbol (lib_id "power:GND") (at 119.38 45.72 270) (unit 1)
     (in_bom yes) (on_board yes)
-    (property "Reference" "#PWR0138" (id 0) (at 113.03 45.72 0)
+    (property "Reference" "#PWR0140" (id 0) (at 113.03 45.72 0)
       (effects (font (size 1.27 1.27)) hide)
     )
@@
   (symbol (lib_id "power:GND") (at 109.22 82.55 0) (unit 1)
     (in_bom yes) (on_board yes)
-    (property "Reference" "#PWR0130" (id 0) (at 109.22 88.9 0)
+    (property "Reference" "#PWR0132" (id 0) (at 109.22 88.9 0)
       (effects (font (size 1.27 1.27)) hide)
     )
@@
   (symbol (lib_id "power:GND") (at 160.02 137.16 90) (mirror x) (unit 1)
     (in_bom yes) (on_board yes) (fields_autoplaced)
-    (property "Reference" "#PWR0145" (id 0) (at 166.37 137.16 0)
+    (property "Reference" "#PWR0147" (id 0) (at 166.37 137.16 0)
       (effects (font (size 1.27 1.27)) hide)
     )
@@
     (property "Datasheet" "74CBTLV3257BQ_115" (id 3) (at 106.68 76.2 0)
       (effects (font (size 1.27 1.27) italic) hide)
+    )
+    (property "MFR" "Nexperia USA" (id 4) (at 127 82.55 0)
+      (effects (font (size 1.27 1.27)) hide)
+    )
+    (property "MFR_PN" "74CBTLV3257BQ,115" (id 5) (at 127 82.55 0)
+      (effects (font (size 1.27 1.27)) hide)
     )
     (pin "1")
@@
   (symbol (lib_id "power:+2V8") (at 111.76 74.93 0) (unit 1)
     (in_bom yes) (on_board yes)
-    (property "Reference" "#PWR0133" (id 0) (at 111.76 78.74 0)
+    (property "Reference" "#PWR0135" (id 0) (at 111.76 78.74 0)
       (effects (font (size 1.27 1.27)) hide)
     )
@@
       (effects (font (size 1.27 1.27)) hide)
     )
+    (property "MFR" "Samsung" (id 4) (at 109.22 80.01 0)
+      (effects (font (size 1.27 1.27)) hide)
+    )
+    (property "MFR_PN" "CL05B104KP5NNNC" (id 5) (at 109.22 80.01 0)
+      (effects (font (size 1.27 1.27)) hide)
+    )
     (pin "1")
     (pin "2")
@@
   (symbol (lib_id "power:GND") (at 160.02 55.88 90) (mirror x) (unit 1)
     (in_bom yes) (on_board yes) (fields_autoplaced)
-    (property "Reference" "#PWR0141" (id 0) (at 166.37 55.88 0)
+    (property "Reference" "#PWR0143" (id 0) (at 166.37 55.88 0)
       (effects (font (size 1.27 1.27)) hide)
     )
@@
       (effects (font (size 1.27 1.27)) hide)
     )
+    (property "MFR" "Samsung" (id 4) (at 109.22 35.56 0)
+      (effects (font (size 1.27 1.27)) hide)
+    )
+    (property "MFR_PN" "CL05B104KP5NNNC" (id 5) (at 109.22 35.56 0)
+      (effects (font (size 1.27 1.27)) hide)
+    )
     (pin "1")
     (pin "2")
@@
   (symbol (lib_id "power:GND") (at 160.02 60.96 90) (mirror x) (unit 1)
     (in_bom yes) (on_board yes) (fields_autoplaced)
-    (property "Reference" "#PWR0143" (id 0) (at 166.37 60.96 0)
+    (property "Reference" "#PWR0145" (id 0) (at 166.37 60.96 0)
       (effects (font (size 1.27 1.27)) hide)
     )
@@
   (symbol (lib_id "power:GND") (at 119.38 90.17 270) (unit 1)
     (in_bom yes) (on_board yes)
-    (property "Reference" "#PWR0139" (id 0) (at 113.03 90.17 0)
+    (property "Reference" "#PWR0141" (id 0) (at 113.03 90.17 0)
       (effects (font (size 1.27 1.27)) hide)
     )
@@
   (symbol (lib_id "power:+2V8") (at 111.76 119.38 0) (unit 1)
     (in_bom yes) (on_board yes)
-    (property "Reference" "#PWR0134" (id 0) (at 111.76 123.19 0)
+    (property "Reference" "#PWR0136" (id 0) (at 111.76 123.19 0)
       (effects (font (size 1.27 1.27)) hide)
     )
@@
   (symbol (lib_id "power:GND") (at 109.22 38.1 0) (unit 1)
     (in_bom yes) (on_board yes)
-    (property "Reference" "#PWR0129" (id 0) (at 109.22 44.45 0)
-      (effects (font (size 1.27 1.27)) hide)
-    )
+    (property "Reference" "#PWR0131" (id 0) (at 109.22 44.45 0)
+      (effects (font (size 1.27 1.27)) hide)
+    )
