File: himax_usb_board/himax_usb_board.kicad_pcb (KiCad board)
At the start: 4 copper layers, 50 x 80 mm, 118 parts, among them J1 USB4105GFA, J2 BM06B-SURS-TF_SWD, SW1 SW_Push, SW2 SW_Push, SW3 SW_Push, U1 STM32F750Z8T6, U10 AP7331-SNG-7, U11 USB3320C-EZK-TR, U12 74CBTLV3257BQ_115, U13 74CBTLV3257BQ_115, U14 74CBTLV3257BQ_115, U2 hm01b0-mwa, U3 HM0360, U4 TL331, U5 74AHC1G08, U6 AP7331-SNG-7, U7 AP7331-SNG-7, U8 AP7331-SNG-7, U9 AP7331-SNG-7, Y1 12MHz

Commit message: hardware wip
Parts:
- added J2: Conn_01x06_Male, Connector_PinHeader_2.54mm:PinHeader_1x06_P2.54mm_Vertical, F.Cu at (2.42, 22.2)
- added R5: 0, Resistor_SMD:R_0402_1005Metric, F.Cu at (12.2, 35.2)
- R6: renamed from R8; value R_Small_US -> 10k
- R7: value R_Small_US -> 330
- R8: renamed from R6; value R_Small_US -> 330
- R9: renamed from R5; value R_Small_US -> 330
- Y1: value 12MHz -> ABM3B-12.000MHZ-B2-T; footprint Crystal:Crystal_SMD_2520-4Pin_2.5x2.0mm -> ABM3B_12_000MHZ_B2_T:XTAL_ABM3B-12.000MHZ-B2-T
- moved R3 26.3 mm to (6.10, 41.5)
- moved R4 24.6 mm to (8.35, 41.5)
- moved R12 15.3 mm to (48.0, 68.0), turned to 0 degrees
- moved R13 12.3 mm to (48.0, 70.4), turned to 0 degrees
- moved R10 11.5 mm to (48.0, 69.2), turned to 0 degrees
- moved C21 6.73 mm to (7.58, 39.2), turned to 180 degrees
- moved FB1 5.76 mm to (9.00, 62.5), turned to 0 degrees
- moved C44 4.59 mm to (32.0, 11.3), turned to 0 degrees
- moved D3 3.95 mm to (2.25, 17.2)
- moved R9 3.95 mm to (2.25, 18.8)
- moved D2 3.72 mm to (2.25, 14.2)
- moved R8 3.72 mm to (2.25, 15.8)
- moved C22 3.58 mm to (8.93, 33.8)
- moved D1 3.53 mm to (2.25, 11.2)
- moved R7 3.53 mm to (2.25, 12.7)
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- renumbered D3 to D1, D1 to D3, J2 to J3, R9 to R10, R10 to R11, R11 to R12, R12 to R13, R13 to R14, R14 to R15, R15 to R16, R16 to R17, R17 to R18, R18 to R19, R19 to R20, R20 to R21, R21 to R22, R22 to R23, R23 to R24, R24 to R25, R25 to R26, R26 to R27, R27 to R28, R28 to R29, R29 to R30, R30 to R31, SW2 to SW1, SW3 to SW2, SW1 to SW3
Connections:
- R6 pad 1: Net-(R8-Pad1) -> /microcontroller/boot0
- R7 pad 1: unconnected-(R7-Pad1) -> Net-(R7-Pad1)
- R8 pad 1: unconnected-(R6-Pad1) -> Net-(R8-Pad1)
- R9 pad 1: unconnected-(R5-Pad1) -> Net-(R9-Pad1)
- SW1 pad 1: Net-(R8-Pad1) -> /microcontroller/boot0
- SW3 pad 1: unconnected-(SW1-Pad1) -> GND
- SW3 pad 2: unconnected-(SW1-Pad2) -> Net-(SW3-Pad2)
- U1 pad 105: unconnected-(U1-Pad105) -> /microcontroller/swdio
- U1 pad 109: unconnected-(U1-Pad109) -> /microcontroller/swdclk
- U1 pad 110: unconnected-(U1-Pad110) -> /microcontroller/3v3_en
- U1 pad 127: /bus mux/camera_select -> unconnected-(U1-Pad127)
- U1 pad 136: unconnected-(U1-Pad136) -> /microcontroller/ulpi_refclk
- U1 pad 138: Net-(R8-Pad1) -> /microcontroller/boot0
- U1 pad 18: unconnected-(U1-Pad18) -> /microcontroller/gpios0
- U1 pad 19: unconnected-(U1-Pad19) -> /microcontroller/gpios1
- U1 pad 20: unconnected-(U1-Pad20) -> /microcontroller/gpios2
- U1 pad 21: unconnected-(U1-Pad21) -> /microcontroller/gpios3
- U1 pad 22: unconnected-(U1-Pad22) -> /microcontroller/gpios4
- U1 pad 23: Net-(C21-Pad2) -> Net-(C22-Pad2)
- U1 pad 24: Net-(C22-Pad2) -> Net-(R5-Pad1)
- U1 pad 34: unconnected-(U1-Pad34) -> /image sensors/hm01b0_int
- U1 pad 35: unconnected-(U1-Pad35) -> /image sensors/hm01b0_trig
- U1 pad 36: /bus mux/camera_data.pclk -> /image sensors/hm01b0_mclk
- U1 pad 42: unconnected-(U1-Pad42) -> /bus mux/camera_data.pclk
- U1 pad 64: unconnected-(U1-Pad64) -> /image sensors/hm0360_mclk
- U1 pad 66: unconnected-(U1-Pad66) -> /image sensors/hm0360_trig
- U1 pad 67: unconnected-(U1-Pad67) -> /image sensors/hm0360_int
- U1 pad 68: unconnected-(U1-Pad68) -> /bus mux/camera_select
- U1 pad 7: unconnected-(U1-Pad7) -> Net-(R7-Pad1)
- U1 pad 75: unconnected-(U1-Pad75) -> Net-(SW3-Pad2)
- U1 pad 77: unconnected-(U1-Pad77) -> /image sensors/hm0360_cfg.clksel
- U1 pad 78: unconnected-(U1-Pad78) -> /image sensors/hm0360_cfg.xshut
- U1 pad 79: unconnected-(U1-Pad79) -> /image sensors/hm0360_cfg.xsleep
- U1 pad 8: unconnected-(U1-Pad8) -> Net-(R8-Pad1)
- U1 pad 9: unconnected-(U1-Pad9) -> Net-(R9-Pad1)
- Y1 pad 2: Net-(C22-Pad2) -> GND
- Y1 pad 3: (no net) -> Net-(C22-Pad2)
- Y1 pad 4: (no net) -> GND
Routing:
- net +2V8: track 196.8 -> 387.4 mm, vias 2 -> 14
- net /image sensors/cameras_i2c.sda: track 0.95 -> 104.0 mm, vias 1 -> 5
- net /image sensors/cameras_i2c.scl: track 1.20 -> 102.1 mm, vias 0 -> 5
- net +1V5: track 4.16 -> 97.2 mm, vias 0 -> 2
- net +1V2: track 0.00 -> 62.7 mm, vias 0 -> 2
- net /image sensors/hm0360_cfg.xsleep: track 0.00 -> 59.5 mm, vias 0 -> 2
- net /microcontroller/~rst: track 0.00 -> 58.9 mm, vias 0 -> 6
- net /image sensors/hm0360_cfg.xshut: track 0.00 -> 58.0 mm, vias 0 -> 2
- net +3V3: track 6.60 -> 64.0 mm, vias 0 -> 3
- net /image sensors/hm0360_cfg.clksel: track 0.00 -> 50.8 mm, vias 0 -> 2
- net /microcontroller/ulpi.clk: track 0.00 -> 48.5 mm, vias 0 -> 2
- net /microcontroller/boot0: track 0.00 -> 48.2 mm, vias 0 -> 2
- net /bus mux/camera_data.d3: track 0.00 -> 46.4 mm, vias 0 -> 2
- net /microcontroller/ulpi.dir: track 0.00 -> 46.1 mm, vias 0 -> 2
- net /bus mux/camera_data.d6: track 0.00 -> 45.8 mm, vias 0 -> 2
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Other:
- board text added: "PF6"
- board text added: "PF7"
- board text added: "PF8"
- board text added: "gnd"
- board text added: "trig_in"
- board text added: "trig_out"
