File: himax_usb_board/himax_usb_board.kicad_sch (KiCad schematic)
At the start: 10 parts

Commit message: schematic wip
Parts:
- removed C? (x2): 47u, symbol Device:C_Small
- removed R? (x2): 10k, symbol Device:R_Small_US
Connections:
- net hm0360_i2c.scl renamed cameras_i2c.scl
- net hm0360_i2c.sda renamed cameras_i2c.sda
- net microcontroller/vusb renamed power/vusb
Other:
- added sheet bus mux (bus_mux.kicad_sch)
- added sheet ulpi (ulpi.kicad_sch)
- sheet image sensors ports: added cameras_i2c{sda scl}, hm01b0_data{d[3..0] hsync vsync pclk int}, hm01b0_int, hm01b0_mclk, hm0360_data{d[7..0] hsync vsync pclk}, hm0360_int, hm0360_strobe; removed hm01b0_data{d[3..0] pclk fvld lvld int}, hm01b0_i2c{sda scl}, hm0360_data{d[7..0] hvld fvld strobe int pclk}, hm0360_i2c{sda scl}
- sheet microcontroller ports: added camera_data{d[7..0] hsync vsync pclk}, cameras_i2c{sda scl}, ulpi_refclk, ulpi{d[7..0] nxt dir stp clk}; removed hm01b0_i2c{sda scl}, hm0360_i2c{sda scl}, usb{d- d+}, vusb
- note removed: "use 1206 cap"
- moved on the sheet: C?, J?, R?

Commit message: board routing wip
Parts:
- removed J?: USB_C_Receptacle_USB2.0, symbol Connector:USB_C_Receptacle_USB2.0
- added J1: USB4105GFA, USB4105_GF_A:GCT_USB4105GFA, symbol USB4105GFA:USB4105GFA
- C1: renamed from C?; footprint (none) -> Capacitor_SMD:C_0603_1608Metric
- R1, R2, R3, R4: renamed from R?; footprint (none) -> Resistor_SMD:R_0402_1005Metric
Connections:
- net GND: now also J1.A1_B12 (GND), J1.B1_A12 (GND__1), J1.SH1 (SHELL_GND), J1.SH2 (SHELL_GND__1), J1.SH3 (SHELL_GND__2), J1.SH4 (SHELL_GND__3)
- net power/vusb: now also J1.A4_B9 (VBUS), J1.B4_A9 (VBUS__1)
- net usb.d+: now also J1.A6 (DP1), J1.B6 (DP2)
- net usb.d-: now also J1.A7 (DN1), J1.B7 (DN2)
- net at R1.2: now also J1.A5 (CC1)
- net at R2.2: now also J1.B5 (CC2)
- no-connect marks 0 -> 3
Other:
- sheet image sensors ports: added hm0360_cfg{clksel xsleep xshut}, hm0360_mclk, hm0360_trig; removed hm0360_strobe
- sheet microcontroller ports: added camera_select, hm01b0_int, hm01b0_mclk, hm01b0_trig, hm0360_cfg{clksel xsleep xshut}, hm0360_int, hm0360_mclk, hm0360_trig; removed none
- moved on the sheet: C1, R1, R2

Commit message: hardware wip
Parts:
- added J2: Conn_01x06_Male, Connector_PinHeader_2.54mm:PinHeader_1x06_P2.54mm_Vertical, symbol Connector:Conn_01x06_Male
- C1: MFR (none) -> Samsung; MFR_PN (none) -> CL10A475KP8NNNC
- J1: MFR (none) -> GCT; MFR_PN (none) -> USB4105-GF-A
- R1, R2: MFR (none) -> Panasonic; MFR_PN (none) -> ERJ-2RKF5101X
- R3, R4: MFR (none) -> Panasonic; MFR_PN (none) -> ERJ-2RKF1002X
Connections:
- net GND: now also J2.6 (Pin_6)
- new net gpios0: J2.1 (Pin_1)
- new net gpios1: J2.2 (Pin_2)
- new net gpios2: J2.3 (Pin_3)
- new net gpios3: J2.4 (Pin_4)
- new net gpios4: J2.5 (Pin_5)
Other:
- sheet microcontroller ports: added gpios[4..0]; removed none
