File: himax_usb_board/image_sensors.kicad_sch (KiCad schematic)
At the start: 24 parts

Commit message: schematic wip
Connections:
- net c+ renamed hm0360_mipi.c+
- net c- renamed hm0360_mipi.c-
- net d+ renamed hm0360_mipi.d+
- net d- renamed hm0360_mipi.d-
- net d0 renamed hm01b0_data.d0
- net hm01b0_data.d0: no longer U?.B1 (D0)
- net d1 renamed hm01b0_data.d1
- net hm01b0_data.d1: no longer U?.A2 (D1)
- net d2 renamed hm01b0_data.d2
- net hm01b0_data.d2: no longer U?.B3 (D2)
- net d3 renamed hm01b0_data.d3
- net hm01b0_data.d3: no longer U?.A3 (D3)
- net d4 renamed hm0360_data.d4
- net d5 renamed hm0360_data.d5
- net d6 renamed hm0360_data.d6
- net d7 renamed hm0360_data.d7
- net fvld renamed hm01b0_data.vsync
- net hm01b0_data.vsync: no longer U?.C3 (FVLD)
- net hvld renamed hm0360_data.hsync
- net int renamed hm01b0_int
- net hm01b0_int: no longer U?.C7 (INT)
- net lvld renamed hm01b0_data.hsync
- net pclk renamed hm01b0_data.pclk
- net hm01b0_data.pclk: no longer U?.B2 (PCLK0)
- net scl renamed cameras_i2c.scl
- net sda renamed cameras_i2c.sda
- net strobe renamed hm0360_strobe
- new net hm0360_data.d0: U?.B1 (D0)
- new net hm0360_data.d1: U?.A2 (D1)
- new net hm0360_data.d2: U?.B3 (D2)
- new net hm0360_data.d3: U?.A3 (D3)
- new net hm0360_data.pclk: U?.B2 (PCLK0)
- new net hm0360_data.vsync: U?.C3 (FVLD)
- new net hm0360_int: U?.C7 (INT)
Other:
- moved on the sheet: C?, FB?, R?, U?

Commit message: board routing wip
Parts:
- added H1, H2: m12_lens_mount_mech, himax:m12_lens_mount_mech, symbol himax:m12_lens_mount_mech
- added R11, R12, R9: 5.1k, Resistor_SMD:R_0402_1005Metric, symbol Device:R_Small_US
- C24, C26, C30, C32: renamed from C?; footprint (none) -> Capacitor_SMD:C_0805_2012Metric
- C25, C27, C28, C29, C31, C33, C34, C35, C36, C37, C38, C39, C40, C41, C42: renamed from C?; footprint (none) -> Capacitor_SMD:C_0402_1005Metric
- FB1, FB2: renamed from FB?; footprint (none) -> Capacitor_SMD:C_0603_1608Metric
- R10: renamed from R?; footprint (none) -> Resistor_SMD:R_0402_1005Metric
- gave numbers to parts that had none: 2
Connections:
- net +2V8: now also U3.E4 (I2C_SEL1), U3.G3 (I2C_SEL0)
- net GND: now also R11.2, R12.2, R9.2
- net hm0360_cfg.clksel: now reaches U3.B5 (CLK_SEL)
- net hm0360_cfg.clksel: now also R11.1
- net hm0360_trig: now reaches U3.D6 (TRIGGER)
- net hm0360_cfg.xshut: now reaches U3.F4 (XSHUTDOWN)
- net hm0360_cfg.xshut: now also R9.1
- net hm0360_mclk: now reaches U3.G1 (MCLK)
- net hm0360_cfg.xsleep: now reaches U3.G4 (XSLEEP)
- net hm0360_cfg.xsleep: now also R12.1
- net hm0360_strobe: no longer names the net of U3.D7 (STROBE)
- no-connect marks 0 -> 4
Other:
- note added: "CXT_SEL pin can float; pulled low internally, anyways, it's a feature that we don't need"
- note added: "FSIN pin floats; unused feature for synchronizing vsync of multiple sensors"
- note added: "METER pin floats; setting can be configured via i2c"
- note added: "STROBE pin is an output nominally for exciting external light sources. We don't need it; let it float."
- note added: "i2c_sel[1..0] = 2'b11 sets i2c addr to 0x35"

Commit message: hardware wip
Parts:
- C24, C26, C30, C32: MFR (none) -> Samsung; MFR_PN (none) -> CL21A106KOQNNNE
- C25, C27, C28, C29, C31, C33, C34, C35, C36, C37, C38, C39, C40, C41, C42: MFR (none) -> Samsung; MFR_PN (none) -> CL05B104KP5NNNC
- FB1, FB2: MFR (none) -> TDK Corporation; MFR_PN (none) -> MPZ1608B471ATA00
- H1, H2: DNP (none) -> DNP; MFR (none) -> N/A; MFR_PN (none) -> N/A
- R10: renamed from R9; MFR (none) -> Panasonic; MFR_PN (none) -> ERJ-2RKF5101X
- R11: renamed from R10; MFR (none) -> Panasonic; MFR_PN (none) -> ERJ-2GE0R00X
- R12: renamed from R11; MFR (none) -> Panasonic; MFR_PN (none) -> ERJ-2RKF5101X
- R13: renamed from R12; MFR (none) -> Panasonic; MFR_PN (none) -> ERJ-2RKF5101X
- U2: MFR (none) -> Himax; MFR_PN (none) -> hm01b0-mwa
- U3: MFR (none) -> Himax; MFR_PN (none) -> HM0360-MWA
