File: himax_usb_board/microcontroller.kicad_sch (KiCad schematic)
At the start: 3 parts

Commit message: schematic wip
Parts:
- removed R?: 3k 1%, symbol Device:R_Small_US
- removed U?: STM32F723ZCTx, Package_QFP:LQFP-144_20x20mm_P0.5mm, symbol MCU_ST_STM32F7:STM32F723ZCTx
- added C? (x15): 100n, symbol Device:C_Small
- added C? (x2): 1u, symbol Device:C_Small
- added C?: 2.2u, symbol Device:C_Small
- added C? (x2): C_Small, symbol Device:C_Small
- added C?: 4.7u, symbol Device:C_Small
- added J?: BM06B-SURS-TF, CONN6x1_BM06B-SURS-TF_JST, symbol BM06B_SURS_TF:BM06B-SURS-TF
- added R?: R_Small_US, symbol Device:R_Small_US
- added SW? (x2): SW_Push, symbol Switch:SW_Push
- added U? (x3): STM32F750Z8T6, LQFP-144_STM, symbol STM32F750Z8T6:STM32F750Z8T6
- added Y?: 12MHz, symbol Device:Crystal
- C?: value C_Small -> 2.2u
Connections:
- net +2V8: now also C?.1, C?.1, C?.1, C?.1, C?.1, C?.1, C?.1, C?.1, C?.1, C?.1, C?.1, C?.1, C?.1, C?.1, C?.1, J?.1, SW?.2, U?.108 (VDD), U?.121 (VDD), U?.131 (VDD), U?.143 (PDR_ON), U?.144 (VDD), U?.17 (VDD), U?.30 (VDD), U?.32 (VREF+), U?.33 (VDDA), U?.39 (VDD), U?.52 (VDD), U?.6 (VBAT), U?.62 (VDD), U?.72 (VDD), U?.84 (VDD)
- net GND: now also C?.2, C?.1, C?.1, C?.2, C?.2, C?.2, C?.2, C?.2, C?.2, C?.2, C?.2, C?.2, C?.2, C?.2, C?.2, C?.2, C?.2, C?.2, C?.2, C?.2, C?.2, C?.2, J?.3, R?.2, SW?.2, U?.107 (VSS), U?.120 (VSS), U?.130 (VSS), U?.16 (VSS), U?.31 (VSSA), U?.38 (VSS), U?.51 (VSS), U?.61 (VSS), U?.83 (VSS), U?.94 (VSS)
- net at C?.1: now also U?.71 (VCAP_1)
- new net: R?.1, SW?.1, U?.138 (BOOT0)
- new net: C?.2, U?.23 (PH0), Y?.1
- new net: C?.2, U?.24 (PH1), Y?.2
- new net: C?.1, U?.106 (VCAP_2)
- new net +3V3: C?.1, C?.1, U?.95 (VDDUSB)
- new net camera_data.d0: U?.96 (PC6)
- new net camera_data.d1: U?.97 (PC7)
- new net camera_data.d2: U?.98 (PC8)
- new net camera_data.d3: U?.99 (PC9)
- new net camera_data.d4: U?.3 (PE4)
- new net camera_data.d5: U?.117 (PD3)
- new net camera_data.d6: U?.4 (PE5)
- new net camera_data.d7: U?.5 (PE6)
- new net camera_data.fvld: U?.124 (PG9)
- new net camera_data.hvld: U?.40 (PA4)
- new net camera_data.pclk: U?.36 (PA2)
- new net cameras_i2c.scl: U?.139 (PB8)
- new net cameras_i2c.sda: U?.137 (PB7)
- new net swdclk: J?.4
- new net swdio: J?.2
- new net swo: J?.5, U?.133 (PB3)
- new net ulpi.clk: U?.41 (PA5)
- new net ulpi.d0: U?.37 (PA3)
- new net ulpi.d1: U?.46 (PB0)
- new net ulpi.d2: U?.47 (PB1)
- new net ulpi.d3: U?.69 (PB10)
- new net ulpi.d4: U?.70 (PB11)
- new net ulpi.d5: U?.73 (PB12)
- new net ulpi.d6: U?.74 (PB13)
- new net ulpi.d7: U?.135 (PB5)
- new net ulpi.dir: U?.28 (PC2)
- new net ulpi.nxt: U?.29 (PC3)
- new net ulpi.stp: U?.26 (PC0)
- new net ~rst: C?.1, J?.6, SW?.1, U?.25 (NRST)
Other:
- note added: "Using a 6-pin JST SUR connector as a programming header. I've designed an adapter board that connects a 10-pin swd connector to one of these connectors."
- moved on the sheet: C?

Commit message: board routing wip
Parts:
- removed J?: BM06B-SURS-TF, CONN6x1_BM06B-SURS-TF_JST, symbol BM06B_SURS_TF:BM06B-SURS-TF
- added D1, D2, D3: LED, LED_SMD:LED_0603_1608Metric, symbol Device:LED
- added J2: BM06B-SURS-TF_SWD, BM06B_SURS_TF:CONN6x1_BM06B-SURS-TF_JST, symbol BM06B_SURS_TF:BM06B-SURS-TF_SWD
- added R5, R6, R7: R_Small_US, Resistor_SMD:R_0402_1005Metric, symbol Device:R_Small_US
- added SW1: SW_Push, himax:TL3302AFxxxQG, symbol Switch:SW_Push
- C10, C11, C12, C13, C14, C15, C16, C17, C18, C19, C20, C21, C22, C23, C5, C6, C7, C8, C9: renamed from C?; footprint (none) -> Capacitor_SMD:C_0402_1005Metric
- C2, C3, C4: renamed from C?; footprint (none) -> Capacitor_SMD:C_0603_1608Metric
- R8: renamed from R?; footprint (none) -> Resistor_SMD:R_0402_1005Metric
- SW2, SW3: renamed from SW?; footprint (none) -> himax:TL3302AFxxxQG
- U1: renamed from U?; footprint LQFP-144_STM -> STM32F750Z8T6:LQFP-144_STM
- Y1: renamed from Y?; footprint (none) -> Crystal:Crystal_SMD_2520-4Pin_2.5x2.0mm
Connections:
- net +2V8: now also J2.1
- net GND: now also D1.1 (K), D2.1 (K), D3.1 (K), J2.3
- net swdclk: now also J2.4
- net swdio: now also J2.2
- net swo: now also J2.5
- net ~rst: now also J2.6
- net camera_select: now reaches U1.127 (PG12)
- net camera_data.fvld renamed camera_data.vsync
- net camera_data.hvld renamed camera_data.hsync
- new net: D3.2 (A), R7.2
- new net: D2.2 (A), R6.2
- new net: D1.2 (A), R5.2
- no-connect marks 0 -> 94
Other:
- note added: "use TL3302AF for switch"

Commit message: hardware wip
Parts:
- removed Y1: 12MHz, Crystal:Crystal_SMD_2520-4Pin_2.5x2.0mm, symbol Device:Crystal
- added R5: 0, Resistor_SMD:R_0402_1005Metric, symbol Device:R_Small_US
- added Y1: ABM3B-12.000MHZ-B2-T, ABM3B_12_000MHZ_B2_T:XTAL_ABM3B-12.000MHZ-B2-T, symbol ABM3B-12.000MHZ-B2-T:ABM3B-12.000MHZ-B2-T
- C10, C12, C13, C14, C15, C16, C17, C18, C19, C20, C23, C5, C6, C7, C9: MFR (none) -> Samsung; MFR_PN (none) -> CL05B104KP5NNNC
- C11, C8: MFR (none) -> Samsung; MFR_PN (none) -> CL05A105KO5NNNC
- C2, C3: MFR (none) -> Samsung; MFR_PN (none) -> CL10A225KP8NNNC
- C21, C22: value C_Small -> 22p; MFR (none) -> Samsung; MFR_PN (none) -> CL05C220JB51PNC
- C4: MFR (none) -> Samsung; MFR_PN (none) -> CL10A475KP8NNNC
- D1: renamed from D3; MFR (none) -> Lite-On; MFR_PN (none) -> LTST-C191KGKT
- D2: MFR (none) -> Lite-On; MFR_PN (none) -> LTST-C191KGKT
- D3: renamed from D1; MFR (none) -> Lite-On; MFR_PN (none) -> LTST-C191KGKT
- J3: renamed from J2; MFR (none) -> JST; MFR_PN (none) -> BM06B-SURS-TF
- R6: renamed from R8; value R_Small_US -> 10k; MFR (none) -> Panasonic; MFR_PN (none) -> ERJ-2RKF1002X
- R7: value R_Small_US -> 330; MFR (none) -> Panasonic; MFR_PN (none) -> ERJ-2RKF3300X
- R8: renamed from R6; value R_Small_US -> 330; MFR (none) -> Panasonic; MFR_PN (none) -> ERJ-2RKF3300X
- R9: renamed from R5; value R_Small_US -> 330; MFR (none) -> Panasonic; MFR_PN (none) -> ERJ-2RKF3300X
- SW1: renamed from SW2; MFR (none) -> E-Switch; MFR_PN (none) -> TL3302AF180QG
- SW2: renamed from SW3; MFR (none) -> E-Switch; MFR_PN (none) -> TL3302AF180QG
- SW3: renamed from SW1; MFR (none) -> E-Switch; MFR_PN (none) -> TL3302AF180QG
- U1: MFR (none) -> STMicroelectronics; MFR_PN (none) -> STM32F750Z8T6
Connections:
- net 3v3_en: now also U1.110 (PA15)
- net GND: now also SW3.1, Y1.2 (GND), Y1.4 (GND__1)
- net camera_data.pclk: now also U1.42 (PA6); no longer U1.36 (PA2)
- net camera_select: now also U1.68 (PE15); no longer U1.127 (PG12)
- net hm01b0_int: now also U1.34 (PA0)
- net hm01b0_mclk: now also U1.36 (PA2)
- net hm01b0_trig: now also U1.35 (PA1)
- net hm0360_int: now also U1.67 (PE14)
- net hm0360_mclk: now also U1.64 (PE11)
- net hm0360_trig: now also U1.66 (PE13)
- net swdclk: now also U1.109 (PA14)
- net swdio: now also U1.105 (PA13)
- net ulpi_refclk: now also U1.136 (PB6)
- net at SW3.2: now also U1.75 (PB14)
- net boot0: now reaches R6.1, SW1.1, U1.138 (BOOT0)
- net at R7.1: now also U1.7 (PC13)
- net gpios0: now reaches U1.18 (PF6)
- net gpios1: now reaches U1.19 (PF7)
- net gpios2: now reaches U1.20 (PF8)
- net gpios3: now reaches U1.21 (PF9)
- net gpios4: now reaches U1.22 (PF10)
- net at U1.23 (PH0): now also C22.2, Y1.3; no longer C21.2
- net at U1.24 (PH1): now also R5.1; no longer C22.2
- net hm0360_cfg.clksel: now reaches U1.77 (PD8)
- net hm0360_cfg.xshut: now reaches U1.78 (PD9)
- net hm0360_cfg.xsleep: now reaches U1.79 (PD10)
- net at U1.8 (PC14): now also R8.1
- net at U1.9 (PC15): now also R9.1
- new net: C21.2, R5.2, Y1.1
- no-connect marks 94 -> 63
Other:
- moved on the sheet: C20, C21, C22, D1, D2, D3, R6, R7, R8, R9, SW1, SW2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
