File: himax_usb_board/power.kicad_sch (KiCad schematic)
At the start: 28 parts

Commit message: board routing wip
Parts:
- added C46, C50: 1u, Capacitor_SMD:C_0402_1005Metric, symbol Device:C_Small
- added R16: 10k, Resistor_SMD:R_0402_1005Metric, symbol Device:R_Small_US
- added R18: 5.6k, Resistor_SMD:R_0402_1005Metric, symbol Device:R_Small_US
- added R19: 1.6k, Resistor_SMD:R_0402_1005Metric, symbol Device:R_Small_US
- added U6: AP7331-SNG-7, diodes_incorporated:DFN200X200X60-8N, symbol diodes_incorporated:AP7331-SNG-7
- C43, C44, C45, C47, C48, C49, C51, C52, C53, C54: renamed from C?; footprint (none) -> Capacitor_SMD:C_0402_1005Metric
- R13, R14, R15, R17, R20, R21, R22, R23, R24, R25, R26, R27: renamed from R?; footprint (none) -> Resistor_SMD:R_0402_1005Metric
- U10, U7, U8, U9: renamed from U?; footprint (none) -> diodes_incorporated:DFN200X200X60-8N
- U5: renamed from U?; footprint (none) -> Package_TO_SOT_SMD:SOT-353_SC-70-5
- gave numbers to parts that had none: 1
Connections:
- net GND: now also U10.7 (GNDPAD1), U10.8 (GNDPAD2), U7.7 (GNDPAD1), U7.8 (GNDPAD2), U8.7 (GNDPAD1), U8.8 (GNDPAD2), U9.7 (GNDPAD1), U9.8 (GNDPAD2), C46.2, C50.2, R19.2, U6.2 (GND), U6.7 (GNDPAD1), U6.8 (GNDPAD2)
- net VCC: now also C43.1, U4.5 (V+), C46.1, R16.2, U6.1 (EN), U6.3 (IN)
- net at U4.4, U5.2: now also R16.1
- new net: R18.2, R19.1, U6.6 (ADJ)
- new net +1V8: C50.1, R18.1, U6.4 (OUT)
Other:
- note added: "1.8v regulator supplies ulpi voltage"
- moved on the sheet: C47, C48, C51, C52, R20, R21, R22, R23, U7, U8

Commit message: hardware wip
Parts:
- C43, C44, C45, C46, C47, C48, C49, C50, C51, C52, C53, C54: MFR (none) -> Samsung; MFR_PN (none) -> CL05A105KO5NNNC
- R14: renamed from R13; MFR (none) -> Panasonic; MFR_PN (none) -> ERJ-2RKF1002X
- R15: renamed from R14; MFR (none) -> Panasonic; MFR_PN (none) -> ERJ-2RKF1002X
- R16: renamed from R15; MFR (none) -> Panasonic; MFR_PN (none) -> ERJ-2RKF1002X
- R17: renamed from R16; MFR (none) -> Panasonic; MFR_PN (none) -> ERJ-2RKF1002X
- R18: renamed from R17; MFR (none) -> Panasonic; MFR_PN (none) -> ERJ-2RKF1002X
- R19: renamed from R18; MFR (none) -> Panasonic; MFR_PN (none) -> ERJ-2RKF5601X
- R20: renamed from R19; MFR (none) -> Panasonic; MFR_PN (none) -> ERJ-2RKF1601X
- R21: renamed from R20; MFR (none) -> Panasonic; MFR_PN (none) -> ERJ-2RKF3301X
- R22: renamed from R21; MFR (none) -> Panasonic; MFR_PN (none) -> ERJ-2RKF1201X
- R23: renamed from R22; MFR (none) -> Panasonic; MFR_PN (none) -> ERJ-2RKF2401X
- R24: renamed from R23; MFR (none) -> Panasonic; MFR_PN (none) -> ERJ-2RKF1201X
- R25: renamed from R24; MFR (none) -> Panasonic; MFR_PN (none) -> ERJ-2RKF1602X
- R26: renamed from R25; MFR (none) -> Panasonic; MFR_PN (none) -> ERJ-2RKF2201X
- R27: renamed from R26; MFR (none) -> Panasonic; MFR_PN (none) -> ERJ-2RKF1202X
- R28: renamed from R27; MFR (none) -> Panasonic; MFR_PN (none) -> ERJ-2RKF2001X
- U10, U6, U7, U8, U9: MFR (none) -> Diodes Incorporated; MFR_PN (none) -> AP7331-SNG-7
- U4: MFR (none) -> Texas Instruments; MFR_PN (none) -> TL331IDBVR
- U5: MFR (none) -> Texas Instruments; MFR_PN (none) -> SN74AHC1G08DCKR
