File: himax_usb_board/ulpi.kicad_sch (KiCad schematic)
At the start: 8 parts

Commit message: board routing wip
Parts:
- C55, C57, C58: renamed from C?; footprint (none) -> Capacitor_SMD:C_0402_1005Metric
- C56: renamed from C?; footprint (none) -> Capacitor_SMD:C_0603_1608Metric
- R28, R29, R30: renamed from R?; footprint (none) -> Resistor_SMD:R_0402_1005Metric
- U11: renamed from U?; footprint USB3320C-EZK-TR:QFN50P500X500X100-33N330X330 -> USB3320C_EZK:QFN50P500X500X100-33N330X330
Connections:
- no-connect marks 0 -> 5

Commit message: hardware wip
Parts:
- C55, C57, C58: MFR (none) -> Samsung; MFR_PN (none) -> CL05B104KP5NNNC
- C56: MFR (none) -> Samsung; MFR_PN (none) -> CL10A225KP8NNNC
- R29: renamed from R28; MFR (none) -> Panasonic; MFR_PN (none) -> ERJ-2RKF1002X
- R30: renamed from R29; MFR (none) -> Panasonic; MFR_PN (none) -> ERJ-2RKF1202X
- R31: renamed from R30; MFR (none) -> Panasonic; MFR_PN (none) -> ERJ-2RKF5101X
- U11: MFR (none) -> Microchip; MFR_PN (none) -> USB3320C-EZK-TR
Changed lines of the file:
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@@
+      (effects (font (size 1.27 1.27)) hide)
+    )
+    (property "MFR" "Samsung" (id 4) (at 168.91 72.39 0)
+      (effects (font (size 1.27 1.27)) hide)
+    )
+    (property "MFR_PN" "CL05B104KP5NNNC" (id 5) (at 168.91 72.39 0)
       (effects (font (size 1.27 1.27)) hide)
     )
@@
   (symbol (lib_id "Device:R_Small_US") (at 105.41 114.3 0) (mirror y) (unit 1)
     (in_bom yes) (on_board yes)
-    (property "Reference" "R28" (id 0) (at 103.759 113.4653 0)
+    (property "Reference" "R29" (id 0) (at 103.759 113.4653 0)
       (effects (font (size 1.27 1.27)) (justify left))
     )
@@
       (effects (font (size 1.27 1.27)) hide)
     )
+    (property "MFR" "Panasonic" (id 4) (at 105.41 114.3 0)
+      (effects (font (size 1.27 1.27)) hide)
+    )
+    (property "MFR_PN" "ERJ-2RKF1002X" (id 5) (at 105.41 114.3 0)
+      (effects (font (size 1.27 1.27)) hide)
+    )
     (pin "1")
     (pin "2")
@@
   (symbol (lib_id "power:+1V8") (at 184.15 67.31 0) (unit 1)
     (in_bom yes) (on_board yes) (fields_autoplaced)
-    (property "Reference" "#PWR0125" (id 0) (at 184.15 71.12 0)
+    (property "Reference" "#PWR0127" (id 0) (at 184.15 71.12 0)
       (effects (font (size 1.27 1.27)) hide)
     )
@@
   (symbol (lib_id "Device:R_Small_US") (at 176.53 116.84 90) (mirror x) (unit 1)
     (in_bom yes) (on_board yes) (fields_autoplaced)
-    (property "Reference" "R30" (id 0) (at 176.53 112.2512 90))
+    (property "Reference" "R31" (id 0) (at 176.53 112.2512 90))
     (property "Value" "5.1k" (id 1) (at 176.53 114.7881 90))
     (property "Footprint" "Resistor_SMD:R_0402_1005Metric" (id 2) (at 176.53 116.84 0)
@@
       (effects (font (size 1.27 1.27)) hide)
     )
+    (property "MFR" "Panasonic" (id 4) (at 176.53 116.84 0)
+      (effects (font (size 1.27 1.27)) hide)
+    )
+    (property "MFR_PN" "ERJ-2RKF5101X" (id 5) (at 176.53 116.84 0)
+      (effects (font (size 1.27 1.27)) hide)
+    )
     (pin "1")
     (pin "2")
@@
   (symbol (lib_id "power:GND") (at 176.53 74.93 0) (mirror y) (unit 1)
     (in_bom yes) (on_board yes)
-    (property "Reference" "#PWR0124" (id 0) (at 176.53 81.28 0)
+    (property "Reference" "#PWR0126" (id 0) (at 176.53 81.28 0)
       (effects (font (size 1.27 1.27)) hide)
     )
@@
   (symbol (lib_id "power:GND") (at 120.65 82.55 0) (mirror y) (unit 1)
     (in_bom yes) (on_board yes)
-    (property "Reference" "#PWR0118" (id 0) (at 120.65 88.9 0)
+    (property "Reference" "#PWR0120" (id 0) (at 120.65 88.9 0)
       (effects (font (size 1.27 1.27)) hide)
     )
@@
   (symbol (lib_id "power:+2V8") (at 193.04 82.55 0) (unit 1)
     (in_bom yes) (on_board yes) (fields_autoplaced)
-    (property "Reference" "#PWR0127" (id 0) (at 193.04 86.36 0)
+    (property "Reference" "#PWR0129" (id 0) (at 193.04 86.36 0)
       (effects (font (size 1.27 1.27)) hide)
     )
@@
   (symbol (lib_id "power:GND") (at 168.91 74.93 0) (mirror y) (unit 1)
     (in_bom yes) (on_board yes)
-    (property "Reference" "#PWR0122" (id 0) (at 168.91 81.28 0)
+    (property "Reference" "#PWR0124" (id 0) (at 168.91 81.28 0)
       (effects (font (size 1.27 1.27)) hide)
     )
@@
     (property "MANUFACTURER" "MICROCHIP" (id 6) (at 143.51 99.06 0)
       (effects (font (size 1.27 1.27)) (justify bottom) hide)
+    )
+    (property "MFR" "Microchip" (id 7) (at 143.51 99.06 0)
+      (effects (font (size 1.27 1.27)) hide)
+    )
+    (property "MFR_PN" "USB3320C-EZK-TR" (id 8) (at 143.51 99.06 0)
+      (effects (font (size 1.27 1.27)) hide)
     )
     (pin "1")
@@
   (symbol (lib_id "power:GND") (at 170.18 134.62 0) (mirror y) (unit 1)
     (in_bom yes) (on_board yes)
-    (property "Reference" "#PWR0123" (id 0) (at 170.18 140.97 0)
+    (property "Reference" "#PWR0125" (id 0) (at 170.18 140.97 0)
       (effects (font (size 1.27 1.27)) hide)
     )
@@
   (symbol (lib_id "power:GND") (at 165.1 129.54 0) (mirror y) (unit 1)
     (in_bom yes) (on_board yes) (fields_autoplaced)
-    (property "Reference" "#PWR0120" (id 0) (at 165.1 135.89 0)
+    (property "Reference" "#PWR0122" (id 0) (at 165.1 135.89 0)
       (effects (font (size 1.27 1.27)) hide)
     )
@@
       (effects (font (size 1.27 1.27)) hide)
     )
+    (property "MFR" "Samsung" (id 4) (at 176.53 72.39 0)
+      (effects (font (size 1.27 1.27)) hide)
+    )
+    (property "MFR_PN" "CL10A225KP8NNNC" (id 5) (at 176.53 72.39 0)
+      (effects (font (size 1.27 1.27)) hide)
+    )
     (pin "1")
     (pin "2")
@@
   (symbol (lib_id "Device:R_Small_US") (at 170.18 129.54 0) (mirror y) (unit 1)
     (in_bom yes) (on_board yes)
-    (property "Reference" "R29" (id 0) (at 168.529 128.7053 0)
+    (property "Reference" "R30" (id 0) (at 168.529 128.7053 0)
       (effects (font (size 1.27 1.27)) (justify left))
     )
@@
       (effects (font (size 1.27 1.27)) hide)
     )
+    (property "MFR" "Panasonic" (id 4) (at 170.18 129.54 0)
+      (effects (font (size 1.27 1.27)) hide)
+    )
+    (property "MFR_PN" "ERJ-2RKF1202X" (id 5) (at 170.18 129.54 0)
+      (effects (font (size 1.27 1.27)) hide)
+    )
     (pin "1")
     (pin "2")
@@
       (effects (font (size 1.27 1.27)) hide)
     )
+    (property "MFR" "Samsung" (id 4) (at 196.85 87.63 0)
+      (effects (font (size 1.27 1.27)) hide)
+    )
+    (property "MFR_PN" "CL05B104KP5NNNC" (id 5) (at 196.85 87.63 0)
+      (effects (font (size 1.27 1.27)) hide)
+    )
     (pin "1")
     (pin "2")
@@
   (symbol (lib_id "power:GND") (at 186.69 74.93 0) (mirror y) (unit 1)
     (in_bom yes) (on_board yes)
-    (property "Reference" "#PWR0126" (id 0) (at 186.69 81.28 0)
+    (property "Reference" "#PWR0128" (id 0) (at 186.69 81.28 0)
       (effects (font (size 1.27 1.27)) hide)
     )
@@
   (symbol (lib_id "power:+2V8") (at 105.41 109.22 0) (unit 1)
     (in_bom yes) (on_board yes) (fields_autoplaced)
-    (property "Reference" "#PWR0117" (id 0) (at 105.41 113.03 0)
+    (property "Reference" "#PWR0119" (id 0) (at 105.41 113.03 0)
       (effects (font (size 1.27 1.27)) hide)
     )
@@
   (symbol (lib_id "power:+3.3V") (at 166.37 67.31 0) (unit 1)
     (in_bom yes) (on_board yes)
-    (property "Reference" "#PWR0121" (id 0) (at 166.37 71.12 0)
+    (property "Reference" "#PWR0123" (id 0) (at 166.37 71.12 0)
       (effects (font (size 1.27 1.27)) hide)
     )
@@
   (symbol (lib_id "power:GND") (at 196.85 90.17 0) (mirror y) (unit 1)
     (in_bom yes) (on_board yes)
-    (property "Reference" "#PWR0128" (id 0) (at 196.85 96.52 0)
+    (property "Reference" "#PWR0130" (id 0) (at 196.85 96.52 0)
       (effects (font (size 1.27 1.27)) hide)
     )
@@
     )
     (property "Datasheet" "~" (id 3) (at 186.69 72.39 0)
+      (effects (font (size 1.27 1.27)) hide)
+    )
+    (property "MFR" "Samsung" (id 4) (at 186.69 72.39 0)
+      (effects (font (size 1.27 1.27)) hide)
+    )
+    (property "MFR_PN" "CL05B104KP5NNNC" (id 5) (at 186.69 72.39 0)
       (effects (font (size 1.27 1.27)) hide)
     )
@@
   (symbol (lib_id "power:+2V8") (at 121.92 73.66 0) (unit 1)
     (in_bom yes) (on_board yes) (fields_autoplaced)
-    (property "Reference" "#PWR0119" (id 0) (at 121.92 77.47 0)
-      (effects (font (size 1.27 1.27)) hide)
-    )
+    (property "Reference" "#PWR0121" (id 0) (at 121.92 77.47 0)
+      (effects (font (size 1.27 1.27)) hide)
+    )
